File: wheatstone_strain_bridge/wheatstone_strain_bridge.kicad_pcb (KiCad board)
At the start: 2 copper layers, 80 x 60 mm, 26 parts, among them J1 Conn_01x04, J10 Conn_01x10, J2 Conn_01x02, J3 Conn_01x04, J4 Conn_01x02, J5 Conn_01x04, J6 Conn_01x02, J7 Conn_01x04, J8 Conn_01x02, J9 Conn_01x10

Commit message: Working on new version with better jumper solution
Parts:
- added J11: Conn_01x02, Pin_Headers:Pin_Header_Straight_1x02, F.Cu at (147.3, 104.1)
- added P1: CONN_01X03, Pin_Headers:Pin_Header_Straight_1x03, F.Cu at (141.6, 81.3)
- added P2: CONN_01X03, Pin_Headers:Pin_Header_Straight_1x03, F.Cu at (149.2, 81.3)
- added P3: CONN_01X03, Pin_Headers:Pin_Header_Straight_1x03, F.Cu at (156.2, 81.3)
- added P4: CONN_01X03, Pin_Headers:Pin_Header_Straight_1x03, F.Cu at (134.0, 81.3)
- added P5: CONN_02X04, Pin_Headers:Pin_Header_Straight_2x04, F.Cu at (-9.00, 35.0)
- added P6: CONN_02X10, Pin_Headers:Pin_Header_Straight_2x10, F.Cu at (85.7, 88.3)
- added P7: CONN_02X14, Pin_Headers:Pin_Header_Straight_2x14, F.Cu at (123.2, 94.6)
- added P8: CONN_01X02, Pin_Headers:Pin_Header_Straight_1x02, F.Cu at (126.4, 87.6)
- added R17: 120, Resistors_SMD:R_1206_HandSoldering, F.Cu at (135.9, 73.7)
- added REF**: 1pin, Connect:1pin, F.Cu at (85.0, 65.0)
- added REF**: 1pin, Connect:1pin, F.Cu at (85.0, 105.0)
- added REF**: 1pin, Connect:1pin, F.Cu at (155.0, 105.0)
- added REF**: 1pin, Connect:1pin, F.Cu at (155.0, 65.0)
- J1, J3, J5, J7: footprint Pin_Headers:Pin_Header_Straight_1x04_Pitch2.54mm -> Pin_Headers:Pin_Header_Straight_1x04
- J10, J9: value Conn_01x10 -> Conn_01x02; footprint Pin_Headers:Pin_Header_Straight_1x10_Pitch2.54mm -> Pin_Headers:Pin_Header_Straight_1x02
- J2, J4, J6, J8: footprint Pin_Headers:Pin_Header_Straight_1x02_Pitch2.54mm -> Pin_Headers:Pin_Header_Straight_1x02
- R1, R10, R11, R12, R13, R14, R15, R16, R2, R3, R4, R5, R6, R7, R8, R9: footprint Resistors_SMD:R_1210_HandSoldering -> Resistors_SMD:R_1206_HandSoldering
- moved R16 273.9 mm to (-119.0, 135.0), turned to 90 degrees
- moved R15 260.3 mm to (-113.0, 135.0), turned to 270 degrees
- moved R14 246.7 mm to (-107.0, 135.0), turned to 270 degrees
- moved R13 233.1 mm to (-101.0, 135.0), turned to 270 degrees
- moved R11 42.6 mm to (119.4, 73.7), turned to 90 degrees
- moved J10 41.5 mm to (138.4, 104.1), turned to 90 degrees
- moved R10 40.8 mm to (104.8, 73.7), turned to 90 degrees
- moved R9 39.3 mm to (89.5, 73.7), turned to 90 degrees
- moved J9 38.9 mm to (120.7, 104.1), turned to 90 degrees
- moved R6 38.6 mm to (123.2, 73.7), turned to 270 degrees
- moved R12 38.4 mm to (153.7, 73.7), turned to 270 degrees
- moved R2 38.2 mm to (93.3, 73.7), turned to 270 degrees
- moved R4 38.1 mm to (108.6, 73.7), turned to 270 degrees
- moved R8 38.1 mm to (148.0, 73.7), turned to 270 degrees
- moved R1 32.7 mm to (97.8, 73.7), turned to 90 degrees
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Connections:
- J10 pad 1: /R_CALIB_4-2 -> /GAUGE_4-5
- J10 pad 2: /R_CALIB_4-1 -> /DC_4-VCC
- J7 pad 1: /GAUGE_4-2 -> /GAUGE_4-8
- J7 pad 4: /MEAS_4-2 -> /GAUGE_4-4
- J8 pad 1: /DC_4-VCC -> /GAUGE_4-1
- J8 pad 2: /GAUGE_4-2 -> /DC_4-GND
- J9 pad 1: /R_CALIB_INPUT-2 -> /GAUGE_4-3
- J9 pad 2: /R_CALIB_INPUT-1 -> /GAUGE_4-4
- R12 pad 1: /DC_4-GND -> /GAUGE_4-4
- R12 pad 2: /GAUGE_4-2 -> Net-(P3-Pad1)
- R7 pad 1: /MEAS_4-2 -> /DC_4-GND
- R7 pad 2: /DC_4-VCC -> Net-(P1-Pad1)
- R8 pad 1: /DC_4-GND -> /DC_4-VCC
- R8 pad 2: /MEAS_4-2 -> Net-(P2-Pad1)
Routing:
- net /GAUGE_4-2: track 97.1 -> 0.00 mm
- net /GAUGE_3-2: track 83.3 -> 5.84 mm
- net /DC_3-VCC: track 80.4 -> 6.66 mm, vias 1 -> 0
- net /DC_2-VCC: track 71.3 -> 7.21 mm, vias 1 -> 0
- net /GAUGE_2-2: track 69.1 -> 5.83 mm
- net /DC_1-VCC: track 64.2 -> 6.90 mm, vias 1 -> 0
- net /DC_4-VCC: track 95.4 -> 40.4 mm, vias 1 -> 0
- net /GAUGE_1-2: track 57.9 -> 6.87 mm
- net /GAUGE_4-4: track 0.00 -> 30.3 mm
- net /GAUGE_4-8: track 0.00 -> 30.0 mm
- net /R_CALIB_INPUT-2: track 27.7 -> 0.00 mm
- net /R_CALIB_INPUT-1: track 25.5 -> 0.00 mm
- net /MEAS_4-2: track 18.0 -> 0.00 mm
- net /R_CALIB_1-1: track 14.1 -> 0.00 mm
- net /DC_1-GND: track 24.5 -> 11.5 mm
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Other:
- board size 80 x 60 mm -> 80 x 50 mm
- board text removed: "1-1"
- board text removed: "1-2"
- board text removed: "2-1"
- board text removed: "2-2"
- board text removed: "3-1"
- board text removed: "3-3"
- board text removed: "4-1"
- board text removed: "4-4"
- board text removed: "CALIBRATION 1"
- board text removed: "CALIBRATION 2"
- board text removed: "Calibration Shunt resistances"
- board text removed: "Connectors to rotary switches"
- board text removed: "DC GND"
- board text removed: "DC VCC"
- board text removed: "MEASURE 1"
- board text removed: "MEASURE 2"
- board text removed: "R 1-1"
- board text removed: "R 1-2"
- board text removed: "R 2-1"
- board text removed: "R 2-2"
- board text removed: "R 3-1"
- board text removed: "R 3-2"
- board text removed: "R 4-1"
- board text removed: "R 4-2"
- board text removed: "Rotary switch config Double pole"
- board text removed: "SG 1-1"
- board text removed: "SG 1-2"
- board text removed: "SG 2-1"
- board text removed: "SG 2-2"
- board text removed: "SG 3-1"
- board text removed: "SG 3-2"
- board text removed: "SG 4-1"
- board text removed: "SG 4-2"
- board text removed: "Wheatstone Bridge Mk. I Pressmaster AB"
